Commit message: feat(lio_sam): update QR detection config and robot frames

File: src/lio_sam/launch/include/config/robot.urdf.xacro (robot description, xacro)
@@ -21,4 +21,16 @@
     <origin xyz="0 0 0" rpy="0 0 0" />
   </joint>
+  <link name="camera_link"></link>
+  <joint name="camera_joint" type="fixed">
+    <parent link="chassis_link" />
+    <child link="camera_link" />
+    <origin xyz="0.12 0.00 0.18" rpy="0 -0.0873 0" />
+  </joint>
+  <link name="camera_color_optical_frame"></link>
+  <joint name="camera_optical_joint" type="fixed">
+    <parent link="camera_link" />
+    <child link="camera_color_optical_frame" />
+    <origin xyz="0 0 0" rpy="-1.57079632679 0 -1.57079632679" />
+  </joint>
   <link name="navsat_link"> </link>
   <joint name="navsat_joint" type="fixed">
